File: TinyWatch/TinyWatch.kicad_pcb (KiCad board)
At the start: 4 copper layers, 40 x 40 mm, 46 parts, among them Q1 NPN, Q2 NPN, U1 ATtiny416-S

Commit message: Started Reworking the Board
Parts:
- removed C1: UPDI, Connector_PinHeader_2.54mm:PinHeader_1x03_P2.54mm_Vertical
- removed Q2: NPN, Package_TO_SOT_SMD:SOT-23
- removed R10, R11, R12, R13, R14, R4, R5, R6, R7, R8, R9: 50, Resistor_SMD:R_0805_2012Metric_Pad1.20x1.40mm_HandSolder
- added J1: DEBUG, Connector_JST:JST_GH_SM05B-GHS-TB_1x05-1MP_P1.25mm_Horizontal, B.Cu at (154.9, 79.2)
- added R2: 50, Resistor_SMD:R_0805_2012Metric_Pad1.20x1.40mm_HandSolder, F.Cu at (156.5, 101.2)
- D1, D10, D11, D12, D13, D14, D15, D16, D17, D18, D2, D22, D23, D24, D3, D4, D5, D6, D7, D8, D9, DM10, DM11, DM12: footprint LED_SMD:LED_0805_2012Metric_Pad1.15x1.40mm_HandSolder -> LED_SMD:LED_0603_1608Metric
- Q1: value NPN -> MMBT5551L
- U1: footprint Package_SO:SOIC-20W_7.5x12.8mm_P1.27mm -> Package_DFN_QFN:QFN-20-1EP_3x3mm_P0.45mm_EP1.6x1.6mm
- moved R3 15.2 mm to (152.0, 101.2), turned to 90 degrees
- moved U1 0.22 mm to (154.8, 95.5), turned to -45 degrees
Connections:
- D1 pad 2: Net-(D1-A) -> LED_H_1
- D10 pad 2: Net-(D10-A) -> LED_H_5
- D11 pad 2: Net-(D11-A) -> LED_H_6
- D12 pad 2: Net-(D11-A) -> LED_H_6
- D13 pad 2: Net-(D13-A) -> LED_H_7
- D14 pad 2: Net-(D13-A) -> LED_H_7
- D15 pad 2: Net-(D15-A) -> LED_H_8
- D16 pad 2: Net-(D15-A) -> LED_H_8
- D17 pad 2: Net-(D17-A) -> LED_H_9
- D18 pad 2: Net-(D17-A) -> LED_H_9
- D2 pad 2: Net-(D1-A) -> LED_H_1
- D22 pad 2: Net-(D22-A) -> LED_H_10
- D23 pad 2: Net-(D23-A) -> LED_H_11
- D24 pad 2: Net-(D24-A) -> LED_H_12
- D3 pad 2: Net-(D3-A) -> LED_H_2
- D4 pad 2: Net-(D3-A) -> LED_H_2
- D5 pad 2: Net-(D5-A) -> LED_H_3
- D6 pad 2: Net-(D5-A) -> LED_H_3
- D7 pad 2: Net-(D7-A) -> LED_H_4
- D8 pad 2: Net-(D7-A) -> LED_H_4
- D9 pad 2: Net-(D10-A) -> LED_H_5
- DM10 pad 2: Net-(D22-A) -> LED_H_10
- DM11 pad 2: Net-(D23-A) -> LED_H_11
- DM12 pad 2: Net-(D24-A) -> LED_H_12
- Q1 pad 1: GS2 -> GND_T_1
- Q1 pad 2: GND_T_1 -> GND
- Q1 pad 3: GND -> unconnected-(Q1-C-Pad3)
- R3 pad 1: LED_H_1 -> GS1
- R3 pad 2: Net-(D1-A) -> unconnected-(R3-Pad2)
- U1 pad 8: Rx -> Net-(U1-PB3)
- U1 pad 9: Tx -> Net-(U1-PB2)
Routing:
- net GS1: track 134.8 -> 0.09 mm, vias 12 -> 0
- net GS2: track 117.5 -> 0.07 mm, vias 12 -> 0
- net Net-(D13-A): track 23.2 -> 0.00 mm
- net GND_T_1: track 20.2 -> 0.00 mm, vias 1 -> 0
- net LED_H_7: track 3.06 -> 23.2 mm
- net Net-(D1-A): track 20.1 -> 0.00 mm
- net GND_T_2: track 19.0 -> 0.00 mm, vias 1 -> 0
- net Net-(D3-A): track 18.5 -> 0.00 mm
- net Net-(D15-A): track 17.3 -> 0.00 mm
- net LED_H_1: track 3.11 -> 20.1 mm
- net BT_Low: track 28.8 -> 12.0 mm
- net LED_H_2: track 2.80 -> 18.5 mm
- net LED_H_8: track 2.39 -> 17.3 mm
- net Net-(D17-A): track 14.3 -> 0.00 mm
- net Net-(D5-A): track 13.0 -> 0.00 mm
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Other:
- board text added: "TinyWatch V2.0"
- board text removed: "TinyWatch V1.0"
