File: TinyWatch/_autosave-TinyWatch.kicad_sch (KiCad schematic)
At the start: 11 parts, among them J1 DEBUG, U1 ATtiny416-S, Y1 Crystal

Commit message: Started Reworking the Board
Other:
- note added: "TP4056"
Changed lines of the file:
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@@
+		)
+	)
+	(text "TP4056"
+		(exclude_from_sim no)
+		(at 77.47 27.178 0)
+		(effects
+			(font
+				(size 1.27 1.27)
+			)
 		)
 	)
