File: TinyWatch/untitled.kicad_sch (KiCad schematic)
At the start: 38 parts, among them Q1 NPN, Q2 NPN

Commit message: Started Reworking the Board
Parts:
- removed Q1, Q2: NPN, Package_TO_SOT_SMD:SOT-23, symbol Simulation_SPICE:NPN
- removed R10, R11, R12, R13, R14, R4, R5, R6, R7, R8, R9: 50, Resistor_SMD:R_0805_2012Metric_Pad1.20x1.40mm_HandSolder, symbol Device:R
- added Q1: MMBT5551L, Package_TO_SOT_SMD:SOT-23, symbol Transistor_BJT:MMBT5551L
- added R2: 50, Resistor_SMD:R_0805_2012Metric_Pad1.20x1.40mm_HandSolder, symbol Device:R
- D1, D10, D11, D12, D13, D14, D15, D16, D17, D18, D2, D22, D23, D24, D3, D4, D5, D6, D7, D8, D9, DM10, DM11, DM12: footprint LED_SMD:LED_0805_2012Metric_Pad1.15x1.40mm_HandSolder -> LED_SMD:LED_0603_1608Metric
Connections:
- net GND: now also Q1.2 (E)
- net GND_T_1: now also Q1.1 (B)
- net GS1: now also R3.1
- net GS2: now also R2.1
- net LED_H_1: now also D1.2 (A), D2.2 (A); no longer R3.1
- net LED_H_10: now also D22.2 (A), DM10.2 (A)
- net LED_H_11: now also D23.2 (A), DM11.2 (A)
- net LED_H_12: now also D24.2 (A), DM12.2 (A)
- net LED_H_2: now also D3.2 (A), D4.2 (A)
- net LED_H_3: now also D5.2 (A), D6.2 (A)
- net LED_H_4: now also D7.2 (A), D8.2 (A)
- net LED_H_5: now also D10.2 (A), D9.2 (A)
- net LED_H_6: now also D11.2 (A), D12.2 (A)
- net LED_H_7: now also D13.2 (A), D14.2 (A)
- net LED_H_8: now also D15.2 (A), D16.2 (A)
- net LED_H_9: now also D17.2 (A), D18.2 (A)
- now unconnected: R3.2
